Commit message: Sensors and Plugins set up

File: description/robot.urdf.xacro (robot description, xacro)
@@ -1,5 +1,5 @@
 <?xml version="1.0"?>
 <robot xmlns:xacro="http://www.ros.org/wiki/xacro" name="robot">
-  <xacro:include filename="robot.gazebo" />
+    <xacro:include filename="robot.gazebo" />
     <xacro:macro name="inertial_box" params="mass x y z *origin">
         <inertial>
@@ -176,3 +176,44 @@
         </xacro:inertial_cylinder>
     </link>
+    <joint name="laser_joint" type="fixed">
+        <parent link="chassis" />
+        <child link="laser_frame" />
+        <origin xyz="-0.055 0 0.08" rpy="0 0 0" />
+    </joint>
+    <link name="laser_frame">
+        <visual>
+            <geometry>
+                <cylinder radius="0.038" length="0.04" />
+            </geometry>
+            <material name="Blue" />
+        </visual>
+        <collision>
+            <geometry>
+                <cylinder radius="0.038" length="0.04" />
+            </geometry>
+        </collision>
+        <xacro:inertial_cylinder mass="0.1" length="0.04" radius="0.038">
+            <origin xyz="0 0 0" rpy="0 0 0" />
+        </xacro:inertial_cylinder>
+    </link>
+    <joint name="camera_joint" type="fixed">
+        <parent link="chassis" />
+        <child link="camera_link" />
+        <origin xyz="0.11 0 0.06" rpy="0 0 0" />
+    </joint>
+    <link name="camera_link">
+        <visual>
+            <origin xyz="-0.0025 0 0.01" />
+            <geometry>
+                <box size="0.005 0.02 0.02" />
+            </geometry>
+            <material name="Red" />
+        </visual>
+    </link>
+    <joint name="camera_optical_joint" type="fixed">
+        <parent link="camera_link" />
+        <child link="camera_link_optical" />
+        <origin xyz="0 0 0" rpy="${-pi/2} 0 ${-pi/2}" />
+    </joint>
+    <link name="camera_link_optical"></link>
 </robot>
